Commit message: Place vehicle parameters in launch file

File: src/ackermann_project/config/ackermann.urdf.xacro (robot description, xacro)
@@ -2,14 +2,23 @@
 <robot name="ackermann" xmlns:xacro="http://ros.org/wiki/xacro">
   <!-- Dimensions taken 2019 from Chevy Cruze https://www.caranddriver.com/chevrolet/cruze/specs -->
+  <!-- Evaluate any parameters passed in and make them properties, which can be used for math operations -->
   <!-- Mass in kilograms -->
-  <xacro:property name="chassis_mass" value="1351" />
-  <xacro:property name="wheel_mass" value="11" />
+  <xacro:arg name="chassis_mass" default="1351" />
+  <xacro:property name="chassis_mass" value="$(arg chassis_mass)" />
+  <xacro:arg name="wheel_mass" default="11" />
+  <xacro:property name="wheel_mass" value="$(arg wheel_mass)" />
   <!-- Length in meters -->
-  <xacro:property name="chassis_length" value="4.45" />
-  <xacro:property name="chassis_width" value="2.7" />
-  <xacro:property name="chassis_height" value="1.45" />
-  <xacro:property name="wheel_radius" value="${0.7112 / 2}" />
-  <xacro:property name="wheel_depth" value="0.2" />
-  <xacro:property name="lon_dist_between_wheels" value="${chassis_length*2/3}" />
+  <xacro:arg name="chassis_length" default="4.45"/>
+  <xacro:property name="chassis_length" value="$(arg chassis_length)" />
+  <xacro:arg name="chassis_width" default="2.7" />
+  <xacro:property name="chassis_width" value="$(arg chassis_width)" />
+  <xacro:arg name="chassis_height" default="1.45" />
+  <xacro:property name="chassis_height" value="$(arg chassis_height)" />
+  <xacro:arg name="wheel_radius" default="0.3556" />
+  <xacro:property name="wheel_radius" value="$(arg wheel_radius)" />
+  <xacro:arg name="wheel_depth" default="0.2" />
+  <xacro:property name="wheel_depth" value="$(arg wheel_depth)" />
+  <xacro:arg name="lon_dist_between_wheels" default="3" />
+  <xacro:property name="lon_dist_between_wheels" value="$(arg lon_dist_between_wheels)" />
   <!-- Material colors -->
   <material name="blue">

Commit message: Pass arguments through

File: src/ackermann_project/config/ackermann.urdf.xacro (robot description, xacro)
@@ -19,6 +19,6 @@
   <xacro:arg name="wheel_depth" default="0.2" />
   <xacro:property name="wheel_depth" value="$(arg wheel_depth)" />
-  <xacro:arg name="lon_dist_between_wheels" default="3" />
-  <xacro:property name="lon_dist_between_wheels" value="$(arg lon_dist_between_wheels)" />
+  <xacro:arg name="wheelbase" default="3" />
+  <xacro:property name="wheelbase" value="$(arg wheelbase)" />
   <!-- Material colors -->
   <material name="blue">
@@ -49,5 +49,5 @@
     <parent link="base_link"/>
     <child link="chassis"/>
-    <origin xyz="${lon_dist_between_wheels/2} 0 ${chassis_height/2}" rpy="0 0 0"/>
+    <origin xyz="${wheelbase/2} 0 ${chassis_height/2}" rpy="0 0 0"/>
     <axis xyz="1 0 0"/>
   </joint>
@@ -118,5 +118,5 @@
         <parent link="chassis"/>
         <child link="${location}_${side}_linkage"/>
-        <origin xyz="${lon_dist_between_wheels*lon/2} ${chassis_width*lat/2} -${chassis_height/2}" rpy="0 0 0"/>
+        <origin xyz="${wheelbase*lon/2} ${chassis_width*lat/2} -${chassis_height/2}" rpy="0 0 0"/>
       </joint>
     </xacro:if>
@@ -126,5 +126,5 @@
         <parent link="chassis"/>
         <child link="${location}_${side}_linkage"/>
-        <origin xyz="${lon_dist_between_wheels*lon/2} ${chassis_width*lat/2} -${chassis_height/2}" rpy="0 0 0"/>
+        <origin xyz="${wheelbase*lon/2} ${chassis_width*lat/2} -${chassis_height/2}" rpy="0 0 0"/>
       </joint>
     </xacro:unless>
@@ -150,5 +150,5 @@
       <wheel_steering_angle_i_gain>0</wheel_steering_angle_i_gain>
       <wheel_steering_angle_d_gain>1e3</wheel_steering_angle_d_gain>
-      <longitudinal_length_between_wheels>${lon_dist_between_wheels}</longitudinal_length_between_wheels>
+      <longitudinal_length_between_wheels>${wheelbase}</longitudinal_length_between_wheels>
       <lateral_width_between_wheels>${chassis_width}</lateral_width_between_wheels>
       <wheel_radius>${wheel_radius}</wheel_radius>

Commit message: Lattice planner (#1)
* Figure out motion primitive math

* Write motion primitive code and test with visualization

* Place vehicle parameters in launch file

* Pass arguments through

* Create utils package

* Add reverse primitives

* Add parameters to launch file

* Add ackermann util files

* AStar ran, not fully debugged

* Turning is working

* Pick angular resolutions

* Add reversing to Astar

* Adjust resolutions

* Add more parameters to launch files

* Clean up code

* Make node index long long int

* Add throw

* Fix collision threshold initialization

* Create ackermann_controller package

File: src/ackermann_project/config/ackermann.urdf.xacro (robot description, xacro)
@@ -2,14 +2,23 @@
 <robot name="ackermann" xmlns:xacro="http://ros.org/wiki/xacro">
   <!-- Dimensions taken 2019 from Chevy Cruze https://www.caranddriver.com/chevrolet/cruze/specs -->
+  <!-- Evaluate any parameters passed in and make them properties, which can be used for math operations -->
   <!-- Mass in kilograms -->
-  <xacro:property name="chassis_mass" value="1351" />
-  <xacro:property name="wheel_mass" value="11" />
+  <xacro:arg name="chassis_mass" default="1351" />
+  <xacro:property name="chassis_mass" value="$(arg chassis_mass)" />
+  <xacro:arg name="wheel_mass" default="11" />
+  <xacro:property name="wheel_mass" value="$(arg wheel_mass)" />
   <!-- Length in meters -->
-  <xacro:property name="chassis_length" value="4.45" />
-  <xacro:property name="chassis_width" value="2.7" />
-  <xacro:property name="chassis_height" value="1.45" />
-  <xacro:property name="wheel_radius" value="${0.7112 / 2}" />
-  <xacro:property name="wheel_depth" value="0.2" />
-  <xacro:property name="lon_dist_between_wheels" value="${chassis_length*2/3}" />
+  <xacro:arg name="chassis_length" default="4.45"/>
+  <xacro:property name="chassis_length" value="$(arg chassis_length)" />
+  <xacro:arg name="chassis_width" default="2.7" />
+  <xacro:property name="chassis_width" value="$(arg chassis_width)" />
+  <xacro:arg name="chassis_height" default="1.45" />
+  <xacro:property name="chassis_height" value="$(arg chassis_height)" />
+  <xacro:arg name="wheel_radius" default="0.3556" />
+  <xacro:property name="wheel_radius" value="$(arg wheel_radius)" />
+  <xacro:arg name="wheel_depth" default="0.2" />
+  <xacro:property name="wheel_depth" value="$(arg wheel_depth)" />
+  <xacro:arg name="wheelbase" default="3" />
+  <xacro:property name="wheelbase" value="$(arg wheelbase)" />
   <!-- Material colors -->
   <material name="blue">
@@ -40,5 +49,5 @@
     <parent link="base_link"/>
     <child link="chassis"/>
-    <origin xyz="${lon_dist_between_wheels/2} 0 ${chassis_height/2}" rpy="0 0 0"/>
+    <origin xyz="${wheelbase/2} 0 ${chassis_height/2}" rpy="0 0 0"/>
     <axis xyz="1 0 0"/>
   </joint>
@@ -109,5 +118,5 @@
         <parent link="chassis"/>
         <child link="${location}_${side}_linkage"/>
-        <origin xyz="${lon_dist_between_wheels*lon/2} ${chassis_width*lat/2} -${chassis_height/2}" rpy="0 0 0"/>
+        <origin xyz="${wheelbase*lon/2} ${chassis_width*lat/2} -${chassis_height/2}" rpy="0 0 0"/>
       </joint>
     </xacro:if>
@@ -117,5 +126,5 @@
         <parent link="chassis"/>
         <child link="${location}_${side}_linkage"/>
-        <origin xyz="${lon_dist_between_wheels*lon/2} ${chassis_width*lat/2} -${chassis_height/2}" rpy="0 0 0"/>
+        <origin xyz="${wheelbase*lon/2} ${chassis_width*lat/2} -${chassis_height/2}" rpy="0 0 0"/>
       </joint>
     </xacro:unless>
@@ -141,5 +150,5 @@
       <wheel_steering_angle_i_gain>0</wheel_steering_angle_i_gain>
       <wheel_steering_angle_d_gain>1e3</wheel_steering_angle_d_gain>
-      <longitudinal_length_between_wheels>${lon_dist_between_wheels}</longitudinal_length_between_wheels>
+      <longitudinal_length_between_wheels>${wheelbase}</longitudinal_length_between_wheels>
       <lateral_width_between_wheels>${chassis_width}</lateral_width_between_wheels>
       <wheel_radius>${wheel_radius}</wheel_radius>

Commit message: Make gazebo ground_truth topic name a parameter

File: src/ackermann_project/config/ackermann.urdf.xacro (robot description, xacro)
@@ -21,4 +21,7 @@
   <xacro:arg name="wheelbase" default="3" />
   <xacro:property name="wheelbase" value="$(arg wheelbase)" />
+  <!-- Topic Names -->
+  <xacro:arg name="vehicle_odom_topic" default="ground_truth" />
+  <xacro:property name="vehicle_odom_topic" value="$(arg vehicle_odom_topic)" />
   <!-- Material colors -->
   <material name="blue">
@@ -154,4 +157,5 @@
       <wheel_radius>${wheel_radius}</wheel_radius>
       <chassis_height>${chassis_height}</chassis_height>
+      <vehicle_odom_topic>${vehicle_odom_topic}</vehicle_odom_topic>
     </plugin>
   </gazebo>

Commit message: Add more parameters to launch file

File: src/ackermann_project/config/ackermann.urdf.xacro (robot description, xacro)
@@ -24,4 +24,6 @@
   <xacro:arg name="vehicle_odom_topic" default="ground_truth" />
   <xacro:property name="vehicle_odom_topic" value="$(arg vehicle_odom_topic)" />
+  <xacro:arg name="vehicle_control_topic" default="cmd_vel" />
+  <xacro:property name="vehicle_control_topic" value="$(arg vehicle_control_topic)" />
   <!-- Material colors -->
   <material name="blue">
@@ -145,5 +147,4 @@
     </plugin>
     <plugin name="ackermann_control_plugin" filename="libAckermannControlPlugin.so">
-      <!-- <chassis>chassis</chassis> -->
       <max_speed>35.7632</max_speed>
       <wheel_angular_velocity_p_gain>1e5</wheel_angular_velocity_p_gain>
@@ -158,4 +159,5 @@
       <chassis_height>${chassis_height}</chassis_height>
       <vehicle_odom_topic>${vehicle_odom_topic}</vehicle_odom_topic>
+      <vehicle_control_topic>${vehicle_control_topic}</vehicle_control_topic>
     </plugin>
   </gazebo>

Commit message: Pure pursuit (#2)
* Make gazebo ground_truth topic name a parameter

* Add more parameters to launch files for pure pursuit

* make C++11 the version

* Add more parameters to launch file

* make parameters dependent on each other

* Create topic for path

* Make path planner a service

* Add vehicle state subscription to planner

* Plan from current vehicle state

* Add visualization of path to RVIZ

* add service file

* Clean up code

* Add dependencies for Goal.srv

* Messy but transform working

* Pure pursuit working basically

* Look for recent transformations to avoid delay in tf

* use variable

* Reduce velocity min velocity error in gazebo controller to get vehicle to stop

* Commend code

* Clean up pure pursuit code

* Clean up and comment A* code

* Make sure pure puruit publishes path updates properly

* Fix pure pursuit erratic steering

File: src/ackermann_project/config/ackermann.urdf.xacro (robot description, xacro)
@@ -21,4 +21,9 @@
   <xacro:arg name="wheelbase" default="3" />
   <xacro:property name="wheelbase" value="$(arg wheelbase)" />
+  <!-- Topic Names -->
+  <xacro:arg name="vehicle_odom_topic" default="ground_truth" />
+  <xacro:property name="vehicle_odom_topic" value="$(arg vehicle_odom_topic)" />
+  <xacro:arg name="vehicle_control_topic" default="cmd_vel" />
+  <xacro:property name="vehicle_control_topic" value="$(arg vehicle_control_topic)" />
   <!-- Material colors -->
   <material name="blue">
@@ -142,5 +147,4 @@
     </plugin>
     <plugin name="ackermann_control_plugin" filename="libAckermannControlPlugin.so">
-      <!-- <chassis>chassis</chassis> -->
       <max_speed>35.7632</max_speed>
       <wheel_angular_velocity_p_gain>1e5</wheel_angular_velocity_p_gain>
@@ -154,4 +158,6 @@
       <wheel_radius>${wheel_radius}</wheel_radius>
       <chassis_height>${chassis_height}</chassis_height>
+      <vehicle_odom_topic>${vehicle_odom_topic}</vehicle_odom_topic>
+      <vehicle_control_topic>${vehicle_control_topic}</vehicle_control_topic>
     </plugin>
   </gazebo>

Commit message: Add steering limit into gazebo plugin

File: src/ackermann_project/config/ackermann.urdf.xacro (robot description, xacro)
@@ -21,4 +21,7 @@
   <xacro:arg name="wheelbase" default="3" />
   <xacro:property name="wheelbase" value="$(arg wheelbase)" />
+  <!-- Limits -->
+  <xacro:arg name="steering_limit_degrees" default="27" />
+  <xacro:property name="steering_limit_degrees" value="$(arg steering_limit_degrees)" />
   <!-- Topic Names -->
   <xacro:arg name="vehicle_odom_topic" default="ground_truth" />
@@ -160,4 +163,5 @@
       <vehicle_odom_topic>${vehicle_odom_topic}</vehicle_odom_topic>
       <vehicle_control_topic>${vehicle_control_topic}</vehicle_control_topic>
+      <steering_limit_degrees>${steering_limit_degrees}</steering_limit_degrees>
     </plugin>
   </gazebo>
